Commit message: added scan + new rosbag

File: src/husky/husky_description/urdf/accessories/sensor_arch.urdf.xacro (robot description, xacro)
@@ -7,5 +7,5 @@
              <visual>
                  <geometry>
-                     <mesh filename="package://husky_description/meshes/accessories/${size}_mm_sensor_arch.dae" />
+                     <!--mesh filename="package://husky_ur3_gazebo/meshes/accessories/${size}_mm_sensor_arch.dae"/-->
                  </geometry>
              </visual>
@@ -13,5 +13,5 @@
                  <origin xyz="0 0 0" rpy="0 0 0"/>
                  <geometry>
-                     <mesh filename="package://husky_description/meshes/accessories/${size}_mm_sensor_arch.dae" />
+                     <!--mesh filename="package://husky_ur3_gazebo/meshes/accessories/${size}_mm_sensor_arch.dae"/-->
                  </geometry>
              </collision>

File: src/husky/husky_description/urdf/husky_macro.urdf.xacro (robot description, xacro)
@@ -17,5 +17,5 @@
   <xacro:include filename="$(find husky_description)/urdf/wheel.urdf.xacro" />
   <xacro:include filename="$(find husky_description)/urdf/accessories/intel_realsense.urdf.xacro"/>
-  <!-- <xacro:include filename="$(find husky_description)/urdf/accessories/sick_lms1xx_mount.urdf.xacro"/> -->
+  <xacro:include filename="$(find husky_description)/urdf/accessories/sick_tim571.urdf.xacro"/>
   <xacro:include filename="$(find husky_description)/urdf/accessories/sensor_arch.urdf.xacro"/>
   <xacro:property name="M_PI" value="3.14159"/>
@@ -89,4 +89,7 @@
       <child link="${prefix}gps_link" />
     </joint>
+    <xacro:sensor_sick_tim571 prefix="front_laser" parent="top_plate_link" prefix_topic="front_laser">
+      <origin xyz="0.35 0.0 0.0" rpy="$(arg laser_rpy)"/>
+    </xacro:sensor_sick_tim571>
     <!-- Husky wheel macros -->
     <xacro:husky_wheel wheel_prefix="${prefix}front_left">
@@ -103,13 +106,4 @@
     </xacro:husky_wheel>
     <xacro:husky_decorate />
-    <!-- <xacro:if value="$(arg laser_enabled)">
-      <xacro:sick_lms1xx_mount prefix="base"/>
-      <xacro:sick_lms1xx frame="base_laser" topic="scan" robot_namespace="$(arg robot_namespace)"/>
-      <joint name="laser_mount_joint" type="fixed">
-        <origin xyz="$(arg laser_xyz)" rpy="$(arg laser_rpy)" />
-        <parent link="top_plate_link" />
-        <child link="base_laser_mount" />
-      </joint>
-    </xacro:if> -->
     <!--
       top sensor arch; include this if we have realsense enabled

File: src/husky/husky_description/urdf/husky_ur3.urdf.xacro (robot description, xacro)
@@ -166,4 +166,7 @@
       <plugin filename="libignition-gazebo-imu-system.so" name="ignition::gazebo::systems::Imu"/>
       <plugin filename="libignition-gazebo-navsat-system.so" name="ignition::gazebo::systems::NavSat"/>
+      <plugin filename="libignition-gazebo-sensors-system.so" name="ignition::gazebo::systems::Sensors">
+        <render_engine>ogre2</render_engine>
+      </plugin>
     </gazebo>
     <!-- IMU Sensor Configuration -->
